Commit message: Model working in RVIZ with mimic joints

File: description/gazebo.xacro (robot description, xacro)
@@ -21,17 +21,3 @@
     <xacro:property name="items" value="${['base_link', 'torso_plate_link', 'right_torso_side_link', 'left_torso_side_link', 'shoulder_cross_link', 'biceps_link']}" />
     <xacro:loop items="${list(items)}"/>
-    <gazebo>
-        <plugin name="gazebo_ros_joint_state_publisher"
-            filename="libgazebo_ros_joint_state_publisher.so">
-            <update_rate>20</update_rate>
-            <joint_name>torso_plate_joint</joint_name>
-            <joint_name>shoulder_joint</joint_name>
-        </plugin>
-    </gazebo>
-    <gazebo>
-        <plugin name="gazebo_ros_joint_pose_trajectory"
-            filename="libgazebo_ros_joint_pose_trajectory.so">
-            <update_rate>20</update_rate>
-        </plugin>
-    </gazebo>
 </robot>

File: description/robot_arm.urdf.xacro (robot description, xacro)
@@ -39,5 +39,5 @@
     <link name="torso_plate_link">
         <visual>
-            <origin xyz="0 0 ${properties['torso']['plate_height'] / 2}" rpy="0 0 ${properties['torso']['upper_limit']}"/>
+            <origin xyz="0 0 ${properties['torso']['plate_height'] / 2}" rpy="0 0 0"/>
             <geometry>
                 <cylinder radius="${properties['torso']['diameter'] / 2}" length="${properties['torso']['plate_height']}"/>
@@ -46,5 +46,5 @@
         </visual>
         <collision>
-            <origin xyz="0 0 ${properties['torso']['plate_height'] / 2}" rpy="0 0 ${properties['torso']['upper_limit']}"/>
+            <origin xyz="0 0 ${properties['torso']['plate_height'] / 2}" rpy="0 0 0"/>
             <geometry>
                 <cylinder radius="${properties['torso']['diameter'] / 2}" length="${properties['torso']['plate_height']}"/>
@@ -52,5 +52,5 @@
         </collision>
         <xacro:inertial_cylinder mass="${properties['torso']['mass']}" length="${properties['torso']['plate_height']}" radius="${properties['torso']['diameter'] / 2}">
-            <origin xyz="0 0 ${properties['torso']['plate_height'] / 2}" rpy="0 0 ${properties['torso']['upper_limit']}"/>
+            <origin xyz="0 0 ${properties['torso']['plate_height'] / 2}" rpy="0 0 0"/>
         </xacro:inertial_cylinder>
     </link>
@@ -153,4 +153,136 @@
         </xacro:inertial_box>
     </link>
+    <!-- Elbow and forearm -->
+    <joint name="elbow_joint" type="revolute">
+        <origin xyz="0 0 ${properties['biceps']['length'] - properties['biceps']['offset']}" rpy="0 0 0"/>
+        <parent link="biceps_link"/>
+        <child link="elbow_mimic_link"/>
+        <axis xyz="1 0 0"/>
+        <limit lower="${properties['forearm']['lower_limit']}" upper="${properties['forearm']['upper_limit']}" velocity="100" effort="100"/>
+    </joint>
+    <link name="elbow_mimic_link">
+        <visual name="">
+            <origin xyz="0 0 0" rpy="0 0 0"/>
+            <geometry>
+                <box size="0 0 0"/>
+            </geometry>
+        </visual>
+        <collision>
+            <origin xyz="0 0 0" rpy="0 0 0"/>
+            <geometry>
+                <box size="0 0 0"/>
+            </geometry>
+        </collision>
+    </link>
+    <joint name="elbow_mimic_joint" type="revolute">
+        <origin xyz="0 0 0" rpy="0 0 0"/>
+        <parent link="elbow_mimic_link"/>
+        <child link="forearm_link"/>
+        <axis xyz="1 0 0"/>
+        <limit lower="${properties['forearm']['lower_limit']}" upper="${properties['forearm']['upper_limit']}" velocity="100" effort="100"/>
+        <mimic joint="shoulder_joint" multiplier="-1.0"/>
+    </joint>
+    <link name="forearm_link">
+        <visual>
+            <origin xyz="0 ${properties['forearm']['length']/2 - properties['forearm']['offset']} 0" rpy="${pi / 2} 0 0"/>
+            <geometry>
+                <box size="${properties['forearm']['width']} ${properties['forearm']['height']} ${properties['forearm']['length']}"/>
+            </geometry>
+            <material name="silver" />
+        </visual>
+        <collision>
+            <origin xyz="0 ${properties['forearm']['length']/2 - properties['forearm']['offset']} 0" rpy="${pi / 2} 0 0"/>
+            <geometry>
+                <box size="${properties['forearm']['width']} ${properties['forearm']['height']} ${properties['forearm']['length']}"/>
+            </geometry>
+        </collision>
+        <xacro:inertial_box mass="${properties['forearm']['mass']}" x="${properties['forearm']['width']}" y="${properties['forearm']['height']}" z="${properties['forearm']['length']}" >
+            <origin xyz="0 ${properties['forearm']['length']/2 - properties['forearm']['offset']} 0" rpy="${pi / 2} 0 0"/>
+        </xacro:inertial_box>
+    </link>
+    <!-- Support Arm -->
+    <joint name="support_arm_cross_joint" type="revolute">
+        <origin xyz="${properties['torso']['side']['offset'] / 2} 0 0 " rpy="0 0 0"/>
+        <parent link="shoulder_cross_link"/>
+        <child link="support_arm_cross_joint_link"/>
+        <axis xyz="1 0 0"/>
+        <limit lower="${properties['support_arm']['crossmember']['lower_limit']}" upper="${properties['support_arm']['crossmember']['upper_limit']}" velocity="100" effort="100"/>
+        <mimic joint="elbow_joint" multiplier="1.0" />
+    </joint>
+    <link name="support_arm_cross_joint_link">
+        <visual>
+            <origin xyz="0 -${properties['support_arm']['crossmember']['length'] / 2} 0" rpy="0 0 ${pi / 2}"/>
+            <geometry>
+                <box size="${properties['support_arm']['crossmember']['length']} ${properties['support_arm']['crossmember']['width']} ${properties['support_arm']['crossmember']['height']}"/>
+            </geometry>
+            <material name="silver" />
+        </visual>
+        <collision>
+            <origin xyz="0 -${properties['support_arm']['crossmember']['length'] / 2} 0" rpy="0 0 ${pi / 2}"/>
+            <geometry>
+                <box size="${properties['support_arm']['crossmember']['length']} ${properties['support_arm']['crossmember']['width']} ${properties['support_arm']['crossmember']['height']}" />
+            </geometry>
+        </collision>
+        <xacro:inertial_box mass="${properties['support_arm']['crossmember']['mass']}" x="${properties['support_arm']['crossmember']['width']}" y="${properties['support_arm']['crossmember']['height']}" z="${properties['support_arm']['crossmember']['length']}" >
+            <origin xyz="0 -${properties['support_arm']['crossmember']['length'] / 2} 0" rpy="0 0 ${pi / 2}"/>
+        </xacro:inertial_box>
+    </link>
+    <joint name="support_elbow_mimic_joint" type="revolute">
+        <origin xyz="0 -${properties['support_arm']['crossmember']['length']} 0" rpy="0 0 0"/>
+        <parent link="support_arm_cross_joint_link"/>
+        <child link="support_arm_connection_link"/>
+        <axis xyz="1 0 0"/>
+        <limit lower="${properties['support_arm']['main']['lower_limit']}" upper="${properties['support_arm']['main']['upper_limit']}" effort="100" velocity="100"/>
+        <mimic joint="elbow_joint" multiplier="-1.0" />
+    </joint>
+    <link name="support_arm_connection_link">
+        <visual>
+            <origin xyz="0 0 0" rpy="0 0 0"/>
+            <geometry>
+                <box size="0 0 0"/>
+            </geometry>
+        </visual>
+        <collision>
+            <origin xyz="0 0 0" rpy="0 0 0"/>
+            <geometry>
+                <box size="0 0 0"/>
+            </geometry>
+        </collision>
+    </link>
+    <joint name="support_shoulder_mimic_joint" type="revolute">
+        <origin xyz="0 0 0" rpy="0 0 0"/>
+        <parent link="support_arm_connection_link"/>
+        <child link="support_arm_link"/>
+        <axis xyz="1 0 0"/>
+        <limit lower="${properties['support_arm']['main']['lower_limit']}" upper="${properties['support_arm']['main']['upper_limit']}" effort="100" velocity="100"/>
+        <mimic joint="shoulder_joint" multiplier="1.0" />
+    </joint>
+    <link name="support_arm_link">
+        <visual>
+            <origin xyz="0 0 ${properties['support_arm']['main']['length'] / 2}" rpy="0 0 0"/>
+            <geometry>
+                <box size="${properties['support_arm']['main']['width']} ${properties['support_arm']['main']['height']} ${properties['support_arm']['main']['length']}"/>
+            </geometry>
+            <material name="silver" />
+        </visual>
+        <collision>
+            <origin xyz="0 0 ${properties['support_arm']['main']['length'] / 2}" rpy="0 0 0"/>
+            <geometry>
+                <box size="${properties['support_arm']['main']['width']} ${properties['support_arm']['main']['height']} ${properties['support_arm']['main']['length']}"/>
+            </geometry>
+        </collision>
+        <xacro:inertial_box mass="${properties['support_arm']['main']['mass']}" x="${properties['support_arm']['main']['width']}" y="${properties['support_arm']['main']['height']}" z="${properties['support_arm']['main']['length']}" >
+            <origin xyz="0 0 ${properties['support_arm']['main']['length'] / 2}" rpy="0 0 0"/>
+        </xacro:inertial_box>
+    </link>
+    <!--<joint name="connection_joint" type="revolute" >
+        <origin xyz="0 0 ${properties['support_arm']['main']['length']}" rpy="0 0 0"/>
+        <parent link="support_arm_link"/>
+        <child link="forearm_link"/>
+        <axis xyz="1 0 0"/>
+        <limit lower="${properties['support_arm']['main']['lower_limit']}" upper="${properties['support_arm']['main']['upper_limit']}" effort="100" velocity="100"/>
+        <mimic joint="shoulder_joint" multiplier="1.0" />
+    </joint> -->
+    <!-- Include custom gazebo configuration to aid when switching from URDF to SDF -->
     <xacro:include filename="gazebo.xacro"/>
 </robot>

Commit message: End of Co-Op term

File: description/gazebo.xacro (robot description, xacro)
@@ -19,5 +19,52 @@
     </xacro:macro>
     <!-- define the list of items to iterate -->
-    <xacro:property name="items" value="${['base_link', 'torso_plate_link', 'right_torso_side_link', 'left_torso_side_link', 'shoulder_cross_link', 'biceps_link']}" />
+    <xacro:property name="items" value="${['base_link', 'plate_link', 'right_side_link', 'left_side_link', 'cross_link', 'biceps_link', 'forearm_link', 'support_brace_link', 'support_arm_link']}" />
     <xacro:loop items="${list(items)}"/>
+    <!-- Configuration for ros2_control with gazebo -->
+    <ros2_control name="RobotArmVisualization" type="system">
+        <hardware>
+            <!-- Hardware interface(s) plugin being loaded -->
+            <plugin>gazebo_ros2_control/GazeboSystem</plugin>
+        </hardware>
+        <!-- List of joints that hardware inerface is talking to in the URDF file -->
+        <joint name="torso_joint">
+            <command_interface name="velocity">
+                <param name="min">-10</param>
+                <param name="max">10</param>
+            </command_interface>
+            <state_interface name="position" />
+        </joint>
+        <joint name="shoulder_joint">
+            <command_interface name="velocity">
+                <param name="min">-10</param>
+                <param name="max">10</param>
+            </command_interface>
+            <state_interface name="position" />
+        </joint>
+        <joint name="elbow_joint">
+            <command_interface name="velocity">
+                <param name="min">-10</param>
+                <param name="max">10</param>
+            </command_interface>
+            <state_interface name="position" />
+        </joint>
+        <joint name="elbow_mimic_joint">
+            <state_interface name="position" />
+        </joint>
+        <joint name="brace_cross_joint">
+            <state_interface name="position" />
+        </joint>
+        <joint name="support_elbow_mimic_joint">
+            <state_interface name="position" />
+        </joint>
+        <joint name="support_shoulder_mimic_joint">
+            <state_interface name="position" />
+        </joint>
+    </ros2_control>
+    <gazebo>
+        <plugin name="gazebo_ros2_control" filename="libgazebo_ros2_control.so">
+            <!-- Load in controllers specified in my_controllers.yaml (Currently causing gzserver to fail when running launch script) -->
+            <!-- <parameters>$(find robot_arm_visualization)/config/my_controllers.yaml</parameters> -->
+        </plugin>
+    </gazebo>
 </robot>

File: description/robot_arm.urdf.xacro (robot description, xacro)
@@ -1,5 +1,4 @@
 <?xml version="1.0"?>
-<robot name="robot_arm"
-    xmlns:xacro="http://www.ros.org/wiki/xacro">
+<robot name="robot_arm" xmlns:xacro="http://www.ros.org/wiki/xacro">
     <xacro:include filename="properties.xacro" />
     <xacro:include filename="macros.xacro" />
@@ -30,12 +29,13 @@
     </link>
     <!-- Rotary torso plate joint to base -->
-    <joint name="torso_plate_joint" type="revolute">
+    <joint name="torso_joint" type="revolute">
         <origin xyz="0 0 ${properties['base']['height'] + 0.01}" rpy="0 0 0"/>
         <parent link="base_link"/>
-        <child link="torso_plate_link"/>
+        <child link="plate_link"/>
         <axis xyz="0 0 1"/>
         <limit lower="${properties['torso']['lower_limit']}" upper="${properties['torso']['upper_limit']}" velocity="100" effort="100"/>
-    </joint>
-    <link name="torso_plate_link">
+        <dynamics damping="10.0" friction="10.0" />
+    </joint>
+    <link name="plate_link">
         <visual>
             <origin xyz="0 0 ${properties['torso']['plate_height'] / 2}" rpy="0 0 0"/>
@@ -58,8 +58,8 @@
     <joint name="right_torso_side_joint" type="fixed">
         <origin xyz="-${properties['torso']['side']['offset']} 0 0" rpy="0 0 0"/>
-        <parent link="torso_plate_link"/>
-        <child link="right_torso_side_link"/>
-    </joint>
-    <link name="right_torso_side_link">
+        <parent link="plate_link"/>
+        <child link="right_side_link"/>
+    </joint>
+    <link name="right_side_link">
         <visual>
             <origin xyz="0 0 ${properties['torso']['side']['height'] / 2}" rpy="0 0 0"/>
@@ -82,8 +82,8 @@
     <joint name="left_torso_side_joint" type="fixed">
         <origin xyz="${properties['torso']['side']['offset']} 0 0" rpy="0 0 0"/>
-        <parent link="torso_plate_link"/>
-        <child link="left_torso_side_link"/>
-    </joint>
-    <link name="left_torso_side_link">
+        <parent link="plate_link"/>
+        <child link="left_side_link"/>
+    </joint>
+    <link name="left_side_link">
         <visual>
             <origin xyz="0 0 ${properties['torso']['side']['height'] / 2}" rpy="0 0 0"/>
@@ -104,10 +104,10 @@
     </link>
     <!-- Shoulder cross member -->
-    <joint name="shoulder_cross_joint" type="fixed">
+    <joint name="cross_joint" type="fixed">
         <origin xyz="-${properties['torso']['side']['offset']} 0 ${properties['shoulder']['crossmember']['height']}" rpy="0 0 0"/>
-        <parent link="torso_plate_link"/>
-        <child link="shoulder_cross_link"/>
-    </joint>
-    <link name="shoulder_cross_link">
+        <parent link="plate_link"/>
+        <child link="cross_link"/>
+    </joint>
+    <link name="cross_link">
         <visual>
             <origin xyz="${properties['shoulder']['crossmember']['length'] / 2} 0 0" rpy="0 ${pi/2} 0"/>
@@ -130,8 +130,9 @@
     <joint name="shoulder_joint" type="revolute">
         <origin xyz="${properties['torso']['side']['offset']} 0 0" rpy="0 0 0"/>
-        <parent link="shoulder_cross_link"/>
+        <parent link="cross_link"/>
         <child link="biceps_link"/>
         <axis xyz="1 0 0"/>
         <limit lower="${properties['shoulder']['lower_limit']}" upper="${properties['shoulder']['upper_limit']}" velocity="100" effort="100"/>
+        <dynamics damping="10.0" friction="10.0" />
     </joint>
     <link name="biceps_link">
@@ -160,4 +161,5 @@
         <axis xyz="1 0 0"/>
         <limit lower="${properties['forearm']['lower_limit']}" upper="${properties['forearm']['upper_limit']}" velocity="100" effort="100"/>
+        <dynamics damping="10.0" friction="10.0" />
     </joint>
     <link name="elbow_mimic_link">
@@ -165,13 +167,16 @@
             <origin xyz="0 0 0" rpy="0 0 0"/>
             <geometry>
-                <box size="0 0 0"/>
-            </geometry>
-        </visual>
-        <collision>
-            <origin xyz="0 0 0" rpy="0 0 0"/>
-            <geometry>
-                <box size="0 0 0"/>
-            </geometry>
-        </collision>
+                <box size="0.001 0.001 0.001"/>
+            </geometry>
+        </visual>
+        <collision>
+            <origin xyz="0 0 0" rpy="0 0 0"/>
+            <geometry>
+                <box size="0.001 0.001 0.001"/>
+            </geometry>
+        </collision>
+        <xacro:inertial_box mass="1" x="0.001" y="0.001" z="0.001" >
+            <origin xyz="0 0 0" rpy="0 0 0"/>
+        </xacro:inertial_box>
     </link>
     <joint name="elbow_mimic_joint" type="revolute">
@@ -182,4 +187,5 @@
         <limit lower="${properties['forearm']['lower_limit']}" upper="${properties['forearm']['upper_limit']}" velocity="100" effort="100"/>
         <mimic joint="shoulder_joint" multiplier="-1.0"/>
+        <dynamics damping="10.0" friction="10.0" />
     </joint>
     <link name="forearm_link">
@@ -202,13 +208,14 @@
     </link>
     <!-- Support Arm -->
-    <joint name="support_arm_cross_joint" type="revolute">
+    <joint name="brace_cross_joint" type="revolute">
         <origin xyz="${properties['torso']['side']['offset'] / 2} 0 0 " rpy="0 0 0"/>
-        <parent link="shoulder_cross_link"/>
-        <child link="support_arm_cross_joint_link"/>
+        <parent link="cross_link"/>
+        <child link="support_brace_link"/>
         <axis xyz="1 0 0"/>
         <limit lower="${properties['support_arm']['crossmember']['lower_limit']}" upper="${properties['support_arm']['crossmember']['upper_limit']}" velocity="100" effort="100"/>
         <mimic joint="elbow_joint" multiplier="1.0" />
-    </joint>
-    <link name="support_arm_cross_joint_link">
+        <dynamics damping="10.0" friction="10.0" />
+    </joint>
+    <link name="support_brace_link">
         <visual>
             <origin xyz="0 -${properties['support_arm']['crossmember']['length'] / 2} 0" rpy="0 0 ${pi / 2}"/>
@@ -230,31 +237,36 @@
     <joint name="support_elbow_mimic_joint" type="revolute">
         <origin xyz="0 -${properties['support_arm']['crossmember']['length']} 0" rpy="0 0 0"/>
-        <parent link="support_arm_cross_joint_link"/>
-        <child link="support_arm_connection_link"/>
+        <parent link="support_brace_link"/>
+        <child link="support_mimic_link"/>
         <axis xyz="1 0 0"/>
         <limit lower="${properties['support_arm']['main']['lower_limit']}" upper="${properties['support_arm']['main']['upper_limit']}" effort="100" velocity="100"/>
         <mimic joint="elbow_joint" multiplier="-1.0" />
-    </joint>
-    <link name="support_arm_connection_link">
-        <visual>
-            <origin xyz="0 0 0" rpy="0 0 0"/>
-            <geometry>
-                <box size="0 0 0"/>
-            </geometry>
-        </visual>
-        <collision>
-            <origin xyz="0 0 0" rpy="0 0 0"/>
-            <geometry>
-                <box size="0 0 0"/>
-            </geometry>
-        </collision>
+        <dynamics damping="10.0" friction="10.0" />
+    </joint>
+    <link name="support_mimic_link">
+        <visual name="">
+            <origin xyz="0 0 0" rpy="0 0 0"/>
+            <geometry>
+                <box size="0.001 0.001 0.001"/>
+            </geometry>
+        </visual>
+        <collision>
+            <origin xyz="0 0 0" rpy="0 0 0"/>
+            <geometry>
+                <box size="0.001 0.001 0.001"/>
+            </geometry>
+        </collision>
+        <xacro:inertial_box mass="1" x="0.001" y="0.001" z="0.001" >
+            <origin xyz="0 0 0" rpy="0 0 0"/>
+        </xacro:inertial_box>
     </link>
     <joint name="support_shoulder_mimic_joint" type="revolute">
         <origin xyz="0 0 0" rpy="0 0 0"/>
-        <parent link="support_arm_connection_link"/>
+        <parent link="support_mimic_link"/>
         <child link="support_arm_link"/>
         <axis xyz="1 0 0"/>
         <limit lower="${properties['support_arm']['main']['lower_limit']}" upper="${properties['support_arm']['main']['upper_limit']}" effort="100" velocity="100"/>
         <mimic joint="shoulder_joint" multiplier="1.0" />
+        <dynamics damping="10.0" friction="10.0" />
     </joint>
     <link name="support_arm_link">
@@ -276,13 +288,5 @@
         </xacro:inertial_box>
     </link>
-    <!--<joint name="connection_joint" type="revolute" >
-        <origin xyz="0 0 ${properties['support_arm']['main']['length']}" rpy="0 0 0"/>
-        <parent link="support_arm_link"/>
-        <child link="forearm_link"/>
-        <axis xyz="1 0 0"/>
-        <limit lower="${properties['support_arm']['main']['lower_limit']}" upper="${properties['support_arm']['main']['upper_limit']}" effort="100" velocity="100"/>
-        <mimic joint="shoulder_joint" multiplier="1.0" />
-    </joint> -->
-    <!-- Include custom gazebo configuration to aid when switching from URDF to SDF -->
+    <!-- Include gazebo configuration to add gazebo properties and configure ros2_control -->
     <xacro:include filename="gazebo.xacro"/>
 </robot>
