Commit message: Restructured

File: visualization_package/description/robot_arm.urdf.xacro (robot description, xacro)
@@ -167,14 +167,14 @@
             <origin xyz="0 0 0" rpy="0 0 0"/>
             <geometry>
-                <box size="0.001 0.001 0.001"/>
-            </geometry>
-        </visual>
-        <collision>
-            <origin xyz="0 0 0" rpy="0 0 0"/>
-            <geometry>
-                <box size="0.001 0.001 0.001"/>
-            </geometry>
-        </collision>
-        <xacro:inertial_box mass="1" x="0.001" y="0.001" z="0.001" >
+                <box size="0 0 0"/>
+            </geometry>
+        </visual>
+        <collision>
+            <origin xyz="0 0 0" rpy="0 0 0"/>
+            <geometry>
+                <box size="0 0 0"/>
+            </geometry>
+        </collision>
+        <xacro:inertial_box mass="1" x="0" y="0" z="0" >
             <origin xyz="0 0 0" rpy="0 0 0"/>
         </xacro:inertial_box>
@@ -248,14 +248,14 @@
             <origin xyz="0 0 0" rpy="0 0 0"/>
             <geometry>
-                <box size="0.001 0.001 0.001"/>
-            </geometry>
-        </visual>
-        <collision>
-            <origin xyz="0 0 0" rpy="0 0 0"/>
-            <geometry>
-                <box size="0.001 0.001 0.001"/>
-            </geometry>
-        </collision>
-        <xacro:inertial_box mass="1" x="0.001" y="0.001" z="0.001" >
+                <box size="0 0 0"/>
+            </geometry>
+        </visual>
+        <collision>
+            <origin xyz="0 0 0" rpy="0 0 0"/>
+            <geometry>
+                <box size="0 0 0"/>
+            </geometry>
+        </collision>
+        <xacro:inertial_box mass="1" x="0" y="0" z="0" >
             <origin xyz="0 0 0" rpy="0 0 0"/>
         </xacro:inertial_box>
